File: eFidget.kicad_pcb (KiCad board)
At the start: 2 copper layers, 99.5 x 72.3 mm, 19 parts, among them SW1 SW_Push, SW2 SW_Push, SW3 SW_Push, SW4 SW_Push, U1 XIAO-RP2040-DIP

Commit message: Update all files with new submission
Parts:
- added D8: 1N5817, Diode_THT:D_DO-41_SOD81_P10.16mm_Horizontal, F.Cu at (202.8, 116.1)
- added J1: Conn_01x01_Pin, Connector_PinHeader_2.54mm:PinHeader_1x01_P2.54mm_Vertical, F.Cu at (209.6, 101.0)
- added J2: Conn_01x01_Pin, Connector_PinHeader_2.54mm:PinHeader_1x01_P2.54mm_Vertical, F.Cu at (209.6, 110.9)
Connections:
- U1 pad 14: unconnected-(U1-VBUS-Pad14) -> Net-(D8-K)
Routing:
- net GND: track 225.4 -> 270.9 mm
- net Net-(D8-K): track 0.00 -> 32.2 mm
- net Net-(D8-A): track 0.00 -> 11.7 mm
